File: AC-K1-v1.kicad_pcb (KiCad board)
At the start: 2 copper layers, 6 parts

Commit message: Worked on spreadsheet
Parts:
- removed REF**: SW_Kailh_Choc_V1V2_5.50u, Switch_Keyboard_Kailh:SW_Kailh_Choc_V1V2_5.50u
- removed REF**: SW_Kailh_Choc_V1V2_ISOEnter, Switch_Keyboard_Kailh:SW_Kailh_Choc_V1V2_ISOEnter
- removed REF**: SW_Kailh_Choc_V1V2_1.75u, Switch_Keyboard_Kailh:SW_Kailh_Choc_V1V2_1.75u
- removed REF**: SW_Kailh_Choc_V1V2_1.25u, Switch_Keyboard_Kailh:SW_Kailh_Choc_V1V2_1.25u
- removed REF**: SW_Kailh_Choc_V1V2_1.50u, Switch_Keyboard_Kailh:SW_Kailh_Choc_V1V2_1.50u
- removed REF**: SW_Kailh_Choc_V1V2_1.00u, Switch_Keyboard_Kailh:SW_Kailh_Choc_V1V2_1.00u

Commit message: Made big part of PCB
Parts:
- added D1: 1N4148, Diode_THT:D_DO-35_SOD27_P7.62mm_Horizontal, B.Cu at (68.5, 71.8)
- added D10: 1N4148, Diode_THT:D_DO-35_SOD27_P7.62mm_Horizontal, B.Cu at (258.5, 71.8)
- added D11: 1N4148, Diode_THT:D_DO-35_SOD27_P7.62mm_Horizontal, B.Cu at (277.5, 71.8)
- added D12: 1N4148, Diode_THT:D_DO-35_SOD27_P7.62mm_Horizontal, B.Cu at (296.5, 71.8)
- added D13: 1N4148, Diode_THT:D_DO-35_SOD27_P7.62mm_Horizontal, B.Cu at (315.5, 71.6)
- added D14: 1N4148, Diode_THT:D_DO-35_SOD27_P7.62mm_Horizontal, B.Cu at (336.5, 79.5)
- added D15: 1N4148, Diode_THT:D_DO-35_SOD27_P7.62mm_Horizontal, B.Cu at (68.5, 92.3)
- added D16: 1N4148, Diode_THT:D_DO-35_SOD27_P7.62mm_Horizontal, B.Cu at (87.5, 92.3)
- added D17: 1N4148, Diode_THT:D_DO-35_SOD27_P7.62mm_Horizontal, B.Cu at (106.5, 92.3)
- added D18: 1N4148, Diode_THT:D_DO-35_SOD27_P7.62mm_Horizontal, B.Cu at (125.5, 92.5)
- added D19: 1N4148, Diode_THT:D_DO-35_SOD27_P7.62mm_Horizontal, B.Cu at (144.5, 92.3)
- added D2: 1N4148, Diode_THT:D_DO-35_SOD27_P7.62mm_Horizontal, B.Cu at (98.0, 71.8)
- added D20: 1N4148, Diode_THT:D_DO-35_SOD27_P7.62mm_Horizontal, B.Cu at (163.5, 92.3)
- added D21: 1N4148, Diode_THT:D_DO-35_SOD27_P7.62mm_Horizontal, B.Cu at (182.5, 92.1)
- added D22: 1N4148, Diode_THT:D_DO-35_SOD27_P7.62mm_Horizontal, B.Cu at (201.5, 92.3)
- added D23: 1N4148, Diode_THT:D_DO-35_SOD27_P7.62mm_Horizontal, B.Cu at (220.5, 92.3)
- added D24: 1N4148, Diode_THT:D_DO-35_SOD27_P7.62mm_Horizontal, B.Cu at (239.5, 92.3)
- added D25: 1N4148, Diode_THT:D_DO-35_SOD27_P7.62mm_Horizontal, B.Cu at (258.5, 92.3)
- added D26: 1N4148, Diode_THT:D_DO-35_SOD27_P7.62mm_Horizontal, B.Cu at (277.5, 92.3)
- added D27: 1N4148, Diode_THT:D_DO-35_SOD27_P7.62mm_Horizontal, B.Cu at (296.5, 92.3)
- added D28: 1N4148, Diode_THT:D_DO-35_SOD27_P7.62mm_Horizontal, B.Cu at (315.5, 92.3)
- added D29: 1N4148, Diode_THT:D_DO-35_SOD27_P7.62mm_Horizontal, B.Cu at (334.5, 92.3)
- added D3: 1N4148, Diode_THT:D_DO-35_SOD27_P7.62mm_Horizontal, B.Cu at (116.5, 71.8)
- added D30: 1N4148, Diode_THT:D_DO-35_SOD27_P7.62mm_Horizontal, B.Cu at (77.5, 111.0)
- added D31: 1N4148, Diode_THT:D_DO-35_SOD27_P7.62mm_Horizontal, B.Cu at (96.5, 111.0)
- added D32: 1N4148, Diode_THT:D_DO-35_SOD27_P7.62mm_Horizontal, B.Cu at (115.5, 111.0)
- added D33: 1N4148, Diode_THT:D_DO-35_SOD27_P7.62mm_Horizontal, B.Cu at (134.5, 110.8)
- added D34: 1N4148, Diode_THT:D_DO-35_SOD27_P7.62mm_Horizontal, B.Cu at (153.5, 110.8)
- added D35: 1N4148, Diode_THT:D_DO-35_SOD27_P7.62mm_Horizontal, B.Cu at (172.5, 110.8)
- added D36: 1N4148, Diode_THT:D_DO-35_SOD27_P7.62mm_Horizontal, B.Cu at (191.5, 110.8)
- added D37: 1N4148, Diode_THT:D_DO-35_SOD27_P7.62mm_Horizontal, B.Cu at (210.5, 110.8)
- added D38: 1N4148, Diode_THT:D_DO-35_SOD27_P7.62mm_Horizontal, B.Cu at (229.5, 110.8)
- added D39: 1N4148, Diode_THT:D_DO-35_SOD27_P7.62mm_Horizontal, B.Cu at (248.5, 110.8)
- added D4: 1N4148, Diode_THT:D_DO-35_SOD27_P7.62mm_Horizontal, B.Cu at (135.5, 71.8)
- added D40: 1N4148, Diode_THT:D_DO-35_SOD27_P7.62mm_Horizontal, B.Cu at (267.5, 110.8)
- added D41: 1N4148, Diode_THT:D_DO-35_SOD27_P7.62mm_Horizontal, B.Cu at (286.5, 110.8)
- added D42: 1N4148, Diode_THT:D_DO-35_SOD27_P7.62mm_Horizontal, B.Cu at (305.5, 110.8)
- added D43: 1N4148, Diode_THT:D_DO-35_SOD27_P7.62mm_Horizontal, B.Cu at (353.5, 110.8)
- added D44: 1N4148, Diode_THT:D_DO-35_SOD27_P7.62mm_Horizontal, B.Cu at (82.0, 129.3)
- added D45: 1N4148, Diode_THT:D_DO-35_SOD27_P7.62mm_Horizontal, B.Cu at (101.0, 129.3)
- added D46: 1N4148, Diode_THT:D_DO-35_SOD27_P7.62mm_Horizontal, B.Cu at (120.0, 129.3)
- added D47: 1N4148, Diode_THT:D_DO-35_SOD27_P7.62mm_Horizontal, B.Cu at (139.0, 129.3)
- added D48: 1N4148, Diode_THT:D_DO-35_SOD27_P7.62mm_Horizontal, B.Cu at (158.0, 129.3)
- added D49: 1N4148, Diode_THT:D_DO-35_SOD27_P7.62mm_Horizontal, B.Cu at (177.0, 129.3)
- added D5: 1N4148, Diode_THT:D_DO-35_SOD27_P7.62mm_Horizontal, B.Cu at (154.5, 71.8)
- added D50: 1N4148, Diode_THT:D_DO-35_SOD27_P7.62mm_Horizontal, B.Cu at (196.0, 129.3)
- added D51: 1N4148, Diode_THT:D_DO-35_SOD27_P7.62mm_Horizontal, B.Cu at (215.0, 129.3)
- added D52: 1N4148, Diode_THT:D_DO-35_SOD27_P7.62mm_Horizontal, B.Cu at (234.0, 129.3)
- added D53: 1N4148, Diode_THT:D_DO-35_SOD27_P7.62mm_Horizontal, B.Cu at (253.0, 129.3)
- added D54: 1N4148, Diode_THT:D_DO-35_SOD27_P7.62mm_Horizontal, B.Cu at (272.0, 129.3)
- added D55: 1N4148, Diode_THT:D_DO-35_SOD27_P7.62mm_Horizontal, B.Cu at (291.0, 129.3)
- added D56: 1N4148, Diode_THT:D_DO-35_SOD27_P7.62mm_Horizontal, B.Cu at (310.5, 128.8)
- added D57: 1N4148, Diode_THT:D_DO-35_SOD27_P7.62mm_Horizontal, B.Cu at (353.5, 129.0)
- added D58: 1N4148, Diode_THT:D_DO-35_SOD27_P7.62mm_Horizontal, B.Cu at (330.5, 119.3)
- added D59: 1N4148, Diode_THT:D_DO-35_SOD27_P7.62mm_Horizontal, B.Cu at (73.2, 147.8)
- added D6: 1N4148, Diode_THT:D_DO-35_SOD27_P7.62mm_Horizontal, B.Cu at (178.0, 71.8)
- added D60: 1N4148, Diode_THT:D_DO-35_SOD27_P7.62mm_Horizontal, B.Cu at (92.5, 147.8)
- added D61: 1N4148, Diode_THT:D_DO-35_SOD27_P7.62mm_Horizontal, B.Cu at (111.5, 147.8)
- added D62: 1N4148, Diode_THT:D_DO-35_SOD27_P7.62mm_Horizontal, B.Cu at (130.5, 147.8)
- added D63: 1N4148, Diode_THT:D_DO-35_SOD27_P7.62mm_Horizontal, B.Cu at (149.5, 147.8)
- added D64: 1N4148, Diode_THT:D_DO-35_SOD27_P7.62mm_Horizontal, B.Cu at (168.5, 147.8)
- added D65: 1N4148, Diode_THT:D_DO-35_SOD27_P7.62mm_Horizontal, B.Cu at (187.5, 148.0)
- added D66: 1N4148, Diode_THT:D_DO-35_SOD27_P7.62mm_Horizontal, B.Cu at (206.5, 147.8)
- added D67: 1N4148, Diode_THT:D_DO-35_SOD27_P7.62mm_Horizontal, B.Cu at (225.5, 147.8)
- added D68: 1N4148, Diode_THT:D_DO-35_SOD27_P7.62mm_Horizontal, B.Cu at (244.5, 147.8)
- added D69: 1N4148, Diode_THT:D_DO-35_SOD27_P7.62mm_Horizontal, B.Cu at (263.5, 148.0)
- added D7: 1N4148, Diode_THT:D_DO-35_SOD27_P7.62mm_Horizontal, B.Cu at (197.0, 71.8)
- added D70: 1N4148, Diode_THT:D_DO-35_SOD27_P7.62mm_Horizontal, B.Cu at (282.5, 147.8)
- added D71: 1N4148, Diode_THT:D_DO-35_SOD27_P7.62mm_Horizontal, B.Cu at (315.5, 147.8)
- added D72: 1N4148, Diode_THT:D_DO-35_SOD27_P7.62mm_Horizontal, B.Cu at (334.5, 147.8)
- added D73: 1N4148, Diode_THT:D_DO-35_SOD27_P7.62mm_Horizontal, B.Cu at (353.5, 147.8)
- added D74: 1N4148, Diode_THT:D_DO-35_SOD27_P7.62mm_Horizontal, B.Cu at (73.2, 166.3)
- added D75: 1N4148, Diode_THT:D_DO-35_SOD27_P7.62mm_Horizontal, B.Cu at (97.0, 166.3)
- added D76: 1N4148, Diode_THT:D_DO-35_SOD27_P7.62mm_Horizontal, B.Cu at (120.5, 166.3)
- added D77: 1N4148, Diode_THT:D_DO-35_SOD27_P7.62mm_Horizontal, B.Cu at (226.0, 166.3)
- added D78: 1N4148, Diode_THT:D_DO-35_SOD27_P7.62mm_Horizontal, B.Cu at (249.5, 166.3)
- added D79: 1N4148, Diode_THT:D_DO-35_SOD27_P7.62mm_Horizontal, B.Cu at (273.0, 166.3)
- added D8: 1N4148, Diode_THT:D_DO-35_SOD27_P7.62mm_Horizontal, B.Cu at (216.0, 71.8)
- added D80: 1N4148, Diode_THT:D_DO-35_SOD27_P7.62mm_Horizontal, B.Cu at (296.5, 166.3)
- added D81: 1N4148, Diode_THT:D_DO-35_SOD27_P7.62mm_Horizontal, B.Cu at (315.5, 166.3)
- added D82: 1N4148, Diode_THT:D_DO-35_SOD27_P7.62mm_Horizontal, B.Cu at (334.5, 166.3)
- added D83: 1N4148, Diode_THT:D_DO-35_SOD27_P7.62mm_Horizontal, B.Cu at (353.5, 166.3)
- added D9: 1N4148, Diode_THT:D_DO-35_SOD27_P7.62mm_Horizontal, B.Cu at (235.0, 71.8)
- added J1: S2B-PH-K-SLFSN, Connector_JST:JST_PH_S2B-PH-K_1x02_P2.00mm_Horizontal, B.Cu at (347.6, 76.0)
- added SW1: ESC, Switch_Keyboard_Kailh:SW_Kailh_Choc_V1V2_1.00u, F.Cu at (59.0, 68.0)
- added SW10: F9, Switch_Keyboard_Kailh:SW_Kailh_Choc_V1V2_1.00u, F.Cu at (249.0, 68.0)
- added SW11: F10, Switch_Keyboard_Kailh:SW_Kailh_Choc_V1V2_1.00u, F.Cu at (268.0, 68.0)
- added SW12: F11, Switch_Keyboard_Kailh:SW_Kailh_Choc_V1V2_1.00u, F.Cu at (287.0, 68.0)
- added SW13: F12, Switch_Keyboard_Kailh:SW_Kailh_Choc_V1V2_1.00u, F.Cu at (306.0, 68.0)
- added SW14: CARET, Switch_Keyboard_Kailh:SW_Kailh_Choc_V1V2_1.00u, F.Cu at (59.0, 88.5)
- added SW15: 1, Switch_Keyboard_Kailh:SW_Kailh_Choc_V1V2_1.00u, F.Cu at (78.0, 88.5)
- added SW16: 2, Switch_Keyboard_Kailh:SW_Kailh_Choc_V1V2_1.00u, F.Cu at (97.0, 88.5)
- added SW17: 3, Switch_Keyboard_Kailh:SW_Kailh_Choc_V1V2_1.00u, F.Cu at (116.0, 88.5)
- added SW18: 4, Switch_Keyboard_Kailh:SW_Kailh_Choc_V1V2_1.00u, F.Cu at (135.0, 88.5)
- added SW19: 5, Switch_Keyboard_Kailh:SW_Kailh_Choc_V1V2_1.00u, F.Cu at (154.0, 88.5)
- added SW2: F1, Switch_Keyboard_Kailh:SW_Kailh_Choc_V1V2_1.00u, F.Cu at (88.0, 68.0)
- added SW20: 6, Switch_Keyboard_Kailh:SW_Kailh_Choc_V1V2_1.00u, F.Cu at (173.0, 88.5)
- added SW21: 7, Switch_Keyboard_Kailh:SW_Kailh_Choc_V1V2_1.00u, F.Cu at (192.0, 88.5)
- added SW22: 8, Switch_Keyboard_Kailh:SW_Kailh_Choc_V1V2_1.00u, F.Cu at (211.0, 88.5)
- added SW23: 9, Switch_Keyboard_Kailh:SW_Kailh_Choc_V1V2_1.00u, F.Cu at (230.0, 88.5)
- added SW24: 0, Switch_Keyboard_Kailh:SW_Kailh_Choc_V1V2_1.00u, F.Cu at (249.0, 88.5)
- added SW25: ß, Switch_Keyboard_Kailh:SW_Kailh_Choc_V1V2_1.00u, F.Cu at (268.0, 88.5)
- added SW26: GRAVE, Switch_Keyboard_Kailh:SW_Kailh_Choc_V1V2_1.00u, F.Cu at (287.0, 88.5)
- added SW27: BSPC, Switch_Keyboard_Kailh:SW_Kailh_Choc_V1V2_1.00u, F.Cu at (306.0, 88.5)
- added SW28: DELETE, Switch_Keyboard_Kailh:SW_Kailh_Choc_V1V2_1.00u, F.Cu at (325.0, 88.5)
- added SW29: HOME, Switch_Keyboard_Kailh:SW_Kailh_Choc_V1V2_1.00u, F.Cu at (344.0, 88.5)
- added SW3: F2, Switch_Keyboard_Kailh:SW_Kailh_Choc_V1V2_1.00u, F.Cu at (107.0, 68.0)
- added SW30: TAB, Switch_Keyboard_Kailh:SW_Kailh_Choc_V1V2_1.50u, F.Cu at (63.5, 107.0)
- added SW31: Q, Switch_Keyboard_Kailh:SW_Kailh_Choc_V1V2_1.00u, F.Cu at (87.0, 107.0)
- added SW32: W, Switch_Keyboard_Kailh:SW_Kailh_Choc_V1V2_1.00u, F.Cu at (106.0, 107.0)
- added SW33: E, Switch_Keyboard_Kailh:SW_Kailh_Choc_V1V2_1.00u, F.Cu at (125.0, 107.0)
- added SW34: R, Switch_Keyboard_Kailh:SW_Kailh_Choc_V1V2_1.00u, F.Cu at (144.0, 107.0)
- added SW35: T, Switch_Keyboard_Kailh:SW_Kailh_Choc_V1V2_1.00u, F.Cu at (163.0, 107.0)
- added SW36: Z, Switch_Keyboard_Kailh:SW_Kailh_Choc_V1V2_1.00u, F.Cu at (182.0, 107.0)
- added SW37: U, Switch_Keyboard_Kailh:SW_Kailh_Choc_V1V2_1.00u, F.Cu at (201.0, 107.0)
- added SW38: I, Switch_Keyboard_Kailh:SW_Kailh_Choc_V1V2_1.00u, F.Cu at (220.0, 107.0)
- added SW39: O, Switch_Keyboard_Kailh:SW_Kailh_Choc_V1V2_1.00u, F.Cu at (239.0, 107.0)
- added SW4: F3, Switch_Keyboard_Kailh:SW_Kailh_Choc_V1V2_1.00u, F.Cu at (126.0, 68.0)
- added SW40: P, Switch_Keyboard_Kailh:SW_Kailh_Choc_V1V2_1.00u, F.Cu at (258.0, 107.0)
- added SW41: Ü, Switch_Keyboard_Kailh:SW_Kailh_Choc_V1V2_1.00u, F.Cu at (277.0, 107.0)
- added SW42: ASTRK, Switch_Keyboard_Kailh:SW_Kailh_Choc_V1V2_1.00u, F.Cu at (296.0, 107.0)
- added SW43: ENTER, Switch_Keyboard_Kailh:SW_Kailh_Choc_V1V2_ISOEnter, F.Cu at (322.2, 115.5)
- added SW44: PG_UP, Switch_Keyboard_Kailh:SW_Kailh_Choc_V1V2_1.00u, F.Cu at (344.0, 107.0)
- added SW45: LCTRL, Switch_Keyboard_Kailh:SW_Kailh_Choc_V1V2_1.75u, F.Cu at (65.8, 125.5)
- added SW46: A, Switch_Keyboard_Kailh:SW_Kailh_Choc_V1V2_1.00u, F.Cu at (91.5, 125.5)
- added SW47: S, Switch_Keyboard_Kailh:SW_Kailh_Choc_V1V2_1.00u, F.Cu at (110.5, 125.5)
- added SW48: D, Switch_Keyboard_Kailh:SW_Kailh_Choc_V1V2_1.00u, F.Cu at (129.5, 125.5)
- added SW49: F, Switch_Keyboard_Kailh:SW_Kailh_Choc_V1V2_1.00u, F.Cu at (148.5, 125.5)
- added SW5: F4, Switch_Keyboard_Kailh:SW_Kailh_Choc_V1V2_1.00u, F.Cu at (145.0, 68.0)
- added SW50: G, Switch_Keyboard_Kailh:SW_Kailh_Choc_V1V2_1.00u, F.Cu at (167.5, 125.5)
- added SW51: H, Switch_Keyboard_Kailh:SW_Kailh_Choc_V1V2_1.00u, F.Cu at (186.5, 125.5)
- added SW52: J, Switch_Keyboard_Kailh:SW_Kailh_Choc_V1V2_1.00u, F.Cu at (205.5, 125.5)
- added SW53: K, Switch_Keyboard_Kailh:SW_Kailh_Choc_V1V2_1.00u, F.Cu at (224.5, 125.5)
- added SW54: L, Switch_Keyboard_Kailh:SW_Kailh_Choc_V1V2_1.00u, F.Cu at (243.5, 125.5)
- added SW55: Ö, Switch_Keyboard_Kailh:SW_Kailh_Choc_V1V2_1.00u, F.Cu at (262.5, 125.5)
- added SW56: Ä, Switch_Keyboard_Kailh:SW_Kailh_Choc_V1V2_1.00u, F.Cu at (281.5, 125.5)
- added SW57: HASH, Switch_Keyboard_Kailh:SW_Kailh_Choc_V1V2_1.00u, F.Cu at (300.5, 125.0)
- added SW58: PG_DN, Switch_Keyboard_Kailh:SW_Kailh_Choc_V1V2_1.00u, F.Cu at (344.0, 125.0)
- added SW59: LSHIFT, Switch_Keyboard_Kailh:SW_Kailh_Choc_V1V2_1.25u, F.Cu at (61.2, 144.0)
- added SW6: F5, Switch_Keyboard_Kailh:SW_Kailh_Choc_V1V2_1.00u, F.Cu at (168.5, 68.0)
- added SW60: LT, Switch_Keyboard_Kailh:SW_Kailh_Choc_V1V2_1.00u, F.Cu at (83.0, 144.0)
- added SW61: Y, Switch_Keyboard_Kailh:SW_Kailh_Choc_V1V2_1.00u, F.Cu at (102.0, 144.0)
- added SW62: X, Switch_Keyboard_Kailh:SW_Kailh_Choc_V1V2_1.00u, F.Cu at (121.0, 144.0)
- added SW63: C, Switch_Keyboard_Kailh:SW_Kailh_Choc_V1V2_1.00u, F.Cu at (140.0, 144.0)
- added SW64: V, Switch_Keyboard_Kailh:SW_Kailh_Choc_V1V2_1.00u, F.Cu at (159.0, 144.0)
- added SW65: B, Switch_Keyboard_Kailh:SW_Kailh_Choc_V1V2_1.00u, F.Cu at (178.0, 144.0)
- added SW66: N, Switch_Keyboard_Kailh:SW_Kailh_Choc_V1V2_1.00u, F.Cu at (197.0, 144.0)
- added SW67: M, Switch_Keyboard_Kailh:SW_Kailh_Choc_V1V2_1.00u, F.Cu at (216.0, 144.0)
- added SW68: COMMA, Switch_Keyboard_Kailh:SW_Kailh_Choc_V1V2_1.00u, F.Cu at (235.0, 144.0)
- added SW69: DOT, Switch_Keyboard_Kailh:SW_Kailh_Choc_V1V2_1.00u, F.Cu at (254.0, 144.0)
- added SW7: F6, Switch_Keyboard_Kailh:SW_Kailh_Choc_V1V2_1.00u, F.Cu at (187.5, 68.0)
- added SW70: MINUS, Switch_Keyboard_Kailh:SW_Kailh_Choc_V1V2_1.00u, F.Cu at (273.0, 144.0)
- added SW71: RSHIFT, Switch_Keyboard_Kailh:SW_Kailh_Choc_V1V2_1.75u, F.Cu at (299.0, 144.0)
- added SW72: UP, Switch_Keyboard_Kailh:SW_Kailh_Choc_V1V2_1.00u, F.Cu at (325.0, 144.0)
- added SW73: END, Switch_Keyboard_Kailh:SW_Kailh_Choc_V1V2_1.00u, F.Cu at (344.0, 144.0)
- added SW74: LCTRL, Switch_Keyboard_Kailh:SW_Kailh_Choc_V1V2_1.25u, F.Cu at (61.2, 162.5)
- added SW75: LCMD, Switch_Keyboard_Kailh:SW_Kailh_Choc_V1V2_1.25u, F.Cu at (85.2, 162.5)
- added SW76: LALT, Switch_Keyboard_Kailh:SW_Kailh_Choc_V1V2_1.25u, F.Cu at (108.8, 162.5)
- added SW77: SPACE, Switch_Keyboard_Kailh:SW_Kailh_Choc_V1V2_5.50u, F.Cu at (173.0, 162.5)
- added SW78: RALT, Switch_Keyboard_Kailh:SW_Kailh_Choc_V1V2_1.25u, F.Cu at (237.8, 162.5)
- added SW79: FN, Switch_Keyboard_Kailh:SW_Kailh_Choc_V1V2_1.25u, F.Cu at (261.2, 162.5)
- added SW8: F7, Switch_Keyboard_Kailh:SW_Kailh_Choc_V1V2_1.00u, F.Cu at (206.5, 68.0)
- added SW80: RCTRL, Switch_Keyboard_Kailh:SW_Kailh_Choc_V1V2_1.25u, F.Cu at (284.8, 162.5)
- added SW81: LEFT, Switch_Keyboard_Kailh:SW_Kailh_Choc_V1V2_1.00u, F.Cu at (306.0, 162.5)
- added SW82: DOWN, Switch_Keyboard_Kailh:SW_Kailh_Choc_V1V2_1.00u, F.Cu at (325.0, 162.5)
- added SW83: RIGHT, Switch_Keyboard_Kailh:SW_Kailh_Choc_V1V2_1.00u, F.Cu at (344.0, 162.5)
- added SW84: Reset, Button_Switch_THT:SW_PUSH_1P1T_6x3.5mm_H4.3_APEM_MJTP1243, F.Cu at (337.8, 76.2)
- added SW9: F8, Switch_Keyboard_Kailh:SW_Kailh_Choc_V1V2_1.00u, F.Cu at (225.5, 68.0)
- added U1: nice_nano, nice-nano-kicad-master:nice_nano, F.Cu at (334.7, 64.8)
Routing:
- net Net-(SW1-A): track 0.00 -> 400.9 mm
- net Net-(D74-K): track 0.00 -> 386.0 mm
- net Net-(SW15-A): track 0.00 -> 373.1 mm
- net Net-(D59-K): track 0.00 -> 368.1 mm
- net Net-(D44-K): track 0.00 -> 350.4 mm
- net Net-(SW16-A): track 0.00 -> 347.1 mm
- net Net-(D30-K): track 0.00 -> 335.3 mm
- net Net-(SW17-A): track 0.00 -> 303.9 mm
- net Net-(D15-K): track 0.00 -> 291.5 mm
- net Net-(SW18-A): track 0.00 -> 284.5 mm
- net Net-(D1-K): track 0.00 -> 274.7 mm
- net Net-(SW20-A): track 0.00 -> 271.1 mm
- net Net-(SW21-A): track 0.00 -> 228.7 mm
- net Net-(SW22-A): track 0.00 -> 206.8 mm
- net Net-(SW23-A): track 0.00 -> 204.0 mm
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Other:
- board outline added: 308 x 121.5 mm
- board text added: "${REFERENCE}"
- board text added: "002"
- board text added: "006"
- board text added: "008"
- board text added: "010"
- board text added: "017"
- board text added: "020"
- board text added: "022"
- board text added: "024"
- board text added: "029"
- board text added: "031"
- board text added: "100"
- board text added: "104"
- board text added: "111"
- board text added: "113"
- board text added: "115"
- board text added: "GND"
- board text added: "RAW"
- board text added: "RST"
- board text added: "VCC"
- board text added: "nice!nano"
