File: AC-K1-v1.kicad_pcb (KiCad board)
At the start: 2 copper layers, 308 x 121.5 mm, 169 parts, among them J1 S2B-PH-K-SLFSN, SW1 ESC, SW10 F9, SW11 F10, SW12 F11, SW13 F12, SW14 CARET, SW15 1, SW16 2, SW17 3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

Commit message: Fixed wire missing
Routing:
- net Net-(SW19-A): track 194.1 -> 258.7 mm
