File: AC-K1-v1.kicad_pcb (KiCad board)
At the start: 2 copper layers, 308 x 121.5 mm, 169 parts, among them J1 S2B-PH-K-SLFSN, SW1 ESC, SW10 F9, SW11 F10, SW12 F11, SW13 F12, SW14 CARET, SW15 1, SW16 2, SW17 3, SW18 4, SW19 5, SW2 F1, SW20 6, SW21 7, SW22 8, SW23 9, SW24 0, SW25 ß, SW26 GRAVE, SW27 BSPC, SW28 DELETE, SW29 HOME, SW3 F2, SW30 TAB, SW31 Q, SW32 W, SW33 E, SW34 R, SW35 T, SW36 Z, SW37 U, SW38 I, SW39 O, SW4 F3, SW40 P, SW41 Ü, SW42 ASTRK, SW43 ENTER, SW44 PG_UP, SW45 LCTRL, SW46 A, SW47 S, SW48 D, SW49 F, SW5 F4, SW50 G, SW51 H, SW52 J, SW53 K, SW54 L, SW55 Ö, SW56 Ä, SW57 HASH, SW58 PG_DN, SW59 LSHIFT, SW6 F5, SW60 LT, SW61 Y, SW62 X, SW63 C, SW64 V, SW65 B, SW66 N, SW67 M, SW68 COMMA, SW69 DOT, SW7 F6, SW70 MINUS, SW71 RSHIFT, SW72 UP, SW73 END, SW74 LCTRL, SW75 LCMD, SW76 LALT, SW77 SPACE, SW78 RALT, SW79 FN, SW8 F7, SW80 RCTRL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

Commit message: Redoing everything
Parts:
- D1, D10, D11, D12, D13, D14, D15, D16, D17, D18, D19, D2, D20, D21, D22, D23, D24, D25, D26, D27, D28, D29, D3, D30, D31, D32, D33, D34, D35, D36, D37, D38, D39, D4, D40, D41, D42, D43, D44, D45, D46, D47, D48, D49, D5, D50, D51, D52, D53, D54, D55, D56, D57, D58, D59, D6, D60, D61, D62, D63, D64, D65, D66, D67, D68, D69, D7, D70, D71, D72, D73, D74, D75, D76, D77, D78, D79, D8, D80, D81, D82, D83, D9, J1: moved to F.Cu
- SW1, SW83: footprint Switch_Keyboard_Kailh:SW_Kailh_Choc_V1V2_1.00u -> marbastlib-choc:SW_choc_v1_1u
- SW10: value F9 -> A; footprint Switch_Keyboard_Kailh:SW_Kailh_Choc_V1V2_1.00u -> marbastlib-choc:SW_choc_v1_1u
- SW11: value F10 -> BSLH; footprint Switch_Keyboard_Kailh:SW_Kailh_Choc_V1V2_1.00u -> marbastlib-choc:SW_choc_v1_1u
- SW12: value F11 -> LCMD; footprint Switch_Keyboard_Kailh:SW_Kailh_Choc_V1V2_1.00u -> marbastlib-choc:SW_choc_v1_1.25u
- SW13: value F12 -> F2; footprint Switch_Keyboard_Kailh:SW_Kailh_Choc_V1V2_1.00u -> marbastlib-choc:SW_choc_v1_1u
- SW14: value CARET -> 2; footprint Switch_Keyboard_Kailh:SW_Kailh_Choc_V1V2_1.00u -> marbastlib-choc:SW_choc_v1_1u
- SW15: value 1 -> W; footprint Switch_Keyboard_Kailh:SW_Kailh_Choc_V1V2_1.00u -> marbastlib-choc:SW_choc_v1_1u
- SW16: value 2 -> S; footprint Switch_Keyboard_Kailh:SW_Kailh_Choc_V1V2_1.00u -> marbastlib-choc:SW_choc_v1_1u
- SW17: value 3 -> Z; footprint Switch_Keyboard_Kailh:SW_Kailh_Choc_V1V2_1.00u -> marbastlib-choc:SW_choc_v1_1u
- SW18: value 4 -> LALT; footprint Switch_Keyboard_Kailh:SW_Kailh_Choc_V1V2_1.00u -> marbastlib-choc:SW_choc_v1_1.25u
- SW19: value 5 -> F3; footprint Switch_Keyboard_Kailh:SW_Kailh_Choc_V1V2_1.00u -> marbastlib-choc:SW_choc_v1_1u
- SW2: value F1 -> GRAVE; footprint Switch_Keyboard_Kailh:SW_Kailh_Choc_V1V2_1.00u -> marbastlib-choc:SW_choc_v1_1u
- SW20: value 6 -> 3; footprint Switch_Keyboard_Kailh:SW_Kailh_Choc_V1V2_1.00u -> marbastlib-choc:SW_choc_v1_1u
- SW21: value 7 -> E; footprint Switch_Keyboard_Kailh:SW_Kailh_Choc_V1V2_1.00u -> marbastlib-choc:SW_choc_v1_1u
- SW22: value 8 -> D; footprint Switch_Keyboard_Kailh:SW_Kailh_Choc_V1V2_1.00u -> marbastlib-choc:SW_choc_v1_1u
- SW23: value 9 -> X; footprint Switch_Keyboard_Kailh:SW_Kailh_Choc_V1V2_1.00u -> marbastlib-choc:SW_choc_v1_1u
- SW24: value 0 -> F4; footprint Switch_Keyboard_Kailh:SW_Kailh_Choc_V1V2_1.00u -> marbastlib-choc:SW_choc_v1_1u
- SW25: value ß -> 4; footprint Switch_Keyboard_Kailh:SW_Kailh_Choc_V1V2_1.00u -> marbastlib-choc:SW_choc_v1_1u
- SW26: value GRAVE -> R; footprint Switch_Keyboard_Kailh:SW_Kailh_Choc_V1V2_1.00u -> marbastlib-choc:SW_choc_v1_1u
- SW27: value BSPC -> F; footprint Switch_Keyboard_Kailh:SW_Kailh_Choc_V1V2_1.00u -> marbastlib-choc:SW_choc_v1_1u
- SW28: value DELETE -> C; footprint Switch_Keyboard_Kailh:SW_Kailh_Choc_V1V2_1.00u -> marbastlib-choc:SW_choc_v1_1u
- SW29: value HOME -> 5; footprint Switch_Keyboard_Kailh:SW_Kailh_Choc_V1V2_1.00u -> marbastlib-choc:SW_choc_v1_1u
- SW3: value F2 -> TAB; footprint Switch_Keyboard_Kailh:SW_Kailh_Choc_V1V2_1.00u -> marbastlib-choc:SW_choc_v1_1.5u
- SW30: value TAB -> T; footprint Switch_Keyboard_Kailh:SW_Kailh_Choc_V1V2_1.50u -> marbastlib-choc:SW_choc_v1_1u
- SW31: value Q -> G; footprint Switch_Keyboard_Kailh:SW_Kailh_Choc_V1V2_1.00u -> marbastlib-choc:SW_choc_v1_1u
- SW32: value W -> V; footprint Switch_Keyboard_Kailh:SW_Kailh_Choc_V1V2_1.00u -> marbastlib-choc:SW_choc_v1_1u
- SW33: value E -> F5; footprint Switch_Keyboard_Kailh:SW_Kailh_Choc_V1V2_1.00u -> marbastlib-choc:SW_choc_v1_1u
- SW34: value R -> 6; footprint Switch_Keyboard_Kailh:SW_Kailh_Choc_V1V2_1.00u -> marbastlib-choc:SW_choc_v1_1u
- SW35: value T -> Y; footprint Switch_Keyboard_Kailh:SW_Kailh_Choc_V1V2_1.00u -> marbastlib-choc:SW_choc_v1_1u
- SW36: value Z -> H; footprint Switch_Keyboard_Kailh:SW_Kailh_Choc_V1V2_1.00u -> marbastlib-choc:SW_choc_v1_1u
- SW37: value U -> B; footprint Switch_Keyboard_Kailh:SW_Kailh_Choc_V1V2_1.00u -> marbastlib-choc:SW_choc_v1_1u
- SW38: value I -> SPACE; footprint Switch_Keyboard_Kailh:SW_Kailh_Choc_V1V2_1.00u -> Switch_Keyboard_Kailh:SW_Kailh_Choc_V1_6.00u
- SW39: value O -> F6; footprint Switch_Keyboard_Kailh:SW_Kailh_Choc_V1V2_1.00u -> marbastlib-choc:SW_choc_v1_1u
- SW4: value F3 -> LCTRL; footprint Switch_Keyboard_Kailh:SW_Kailh_Choc_V1V2_1.00u -> marbastlib-choc:SW_choc_v1_1.75u
- SW40: value P -> 7; footprint Switch_Keyboard_Kailh:SW_Kailh_Choc_V1V2_1.00u -> marbastlib-choc:SW_choc_v1_1u
- SW41: value Ü -> U; footprint Switch_Keyboard_Kailh:SW_Kailh_Choc_V1V2_1.00u -> marbastlib-choc:SW_choc_v1_1u
- SW42: value ASTRK -> J; footprint Switch_Keyboard_Kailh:SW_Kailh_Choc_V1V2_1.00u -> marbastlib-choc:SW_choc_v1_1u
- SW43: value ENTER -> N; footprint Switch_Keyboard_Kailh:SW_Kailh_Choc_V1V2_ISOEnter -> marbastlib-choc:SW_choc_v1_1u
- SW44: value PG_UP -> F7; footprint Switch_Keyboard_Kailh:SW_Kailh_Choc_V1V2_1.00u -> marbastlib-choc:SW_choc_v1_1u
- SW45: value LCTRL -> 8; footprint Switch_Keyboard_Kailh:SW_Kailh_Choc_V1V2_1.75u -> marbastlib-choc:SW_choc_v1_1u
- SW46: value A -> I; footprint Switch_Keyboard_Kailh:SW_Kailh_Choc_V1V2_1.00u -> marbastlib-choc:SW_choc_v1_1u
- SW47: value S -> K; footprint Switch_Keyboard_Kailh:SW_Kailh_Choc_V1V2_1.00u -> marbastlib-choc:SW_choc_v1_1u
- SW48: value D -> M; footprint Switch_Keyboard_Kailh:SW_Kailh_Choc_V1V2_1.00u -> marbastlib-choc:SW_choc_v1_1u
- SW49: value F -> F8; footprint Switch_Keyboard_Kailh:SW_Kailh_Choc_V1V2_1.00u -> marbastlib-choc:SW_choc_v1_1u
- SW5: value F4 -> LSHIFT; footprint Switch_Keyboard_Kailh:SW_Kailh_Choc_V1V2_1.00u -> marbastlib-choc:SW_choc_v1_1.25u
- SW50: value G -> 9; footprint Switch_Keyboard_Kailh:SW_Kailh_Choc_V1V2_1.00u -> marbastlib-choc:SW_choc_v1_1u
- SW51: value H -> O; footprint Switch_Keyboard_Kailh:SW_Kailh_Choc_V1V2_1.00u -> marbastlib-choc:SW_choc_v1_1u
- SW52: value J -> L; footprint Switch_Keyboard_Kailh:SW_Kailh_Choc_V1V2_1.00u -> marbastlib-choc:SW_choc_v1_1u
- SW53: value K -> COMMA; footprint Switch_Keyboard_Kailh:SW_Kailh_Choc_V1V2_1.00u -> marbastlib-choc:SW_choc_v1_1u
- SW54: value L -> RALT; footprint Switch_Keyboard_Kailh:SW_Kailh_Choc_V1V2_1.00u -> marbastlib-choc:SW_choc_v1_1.25u
- SW55: value Ö -> F9; footprint Switch_Keyboard_Kailh:SW_Kailh_Choc_V1V2_1.00u -> marbastlib-choc:SW_choc_v1_1u
- SW56: value Ä -> 0; footprint Switch_Keyboard_Kailh:SW_Kailh_Choc_V1V2_1.00u -> marbastlib-choc:SW_choc_v1_1u
- SW57: value HASH -> P; footprint Switch_Keyboard_Kailh:SW_Kailh_Choc_V1V2_1.00u -> marbastlib-choc:SW_choc_v1_1u
- SW58: value PG_DN -> SEMI; footprint Switch_Keyboard_Kailh:SW_Kailh_Choc_V1V2_1.00u -> marbastlib-choc:SW_choc_v1_1u
- SW59: value LSHIFT -> DOT; footprint Switch_Keyboard_Kailh:SW_Kailh_Choc_V1V2_1.25u -> marbastlib-choc:SW_choc_v1_1u
- SW6: value F5 -> LCTRL; footprint Switch_Keyboard_Kailh:SW_Kailh_Choc_V1V2_1.00u -> marbastlib-choc:SW_choc_v1_1.25u
- SW60: value LT -> FN; footprint Switch_Keyboard_Kailh:SW_Kailh_Choc_V1V2_1.00u -> marbastlib-choc:SW_choc_v1_1.25u
- SW61: value Y -> F10; footprint Switch_Keyboard_Kailh:SW_Kailh_Choc_V1V2_1.00u -> marbastlib-choc:SW_choc_v1_1u
- SW62: value X -> MINUS; footprint Switch_Keyboard_Kailh:SW_Kailh_Choc_V1V2_1.00u -> marbastlib-choc:SW_choc_v1_1u
- SW63: value C -> LBKT; footprint Switch_Keyboard_Kailh:SW_Kailh_Choc_V1V2_1.00u -> marbastlib-choc:SW_choc_v1_1u
- SW64: value V -> SQT; footprint Switch_Keyboard_Kailh:SW_Kailh_Choc_V1V2_1.00u -> marbastlib-choc:SW_choc_v1_1u
- SW65: value B -> FSLH; footprint Switch_Keyboard_Kailh:SW_Kailh_Choc_V1V2_1.00u -> marbastlib-choc:SW_choc_v1_1u
- SW66: value N -> RCTRL; footprint Switch_Keyboard_Kailh:SW_Kailh_Choc_V1V2_1.00u -> marbastlib-choc:SW_choc_v1_1.25u
- SW67: value M -> F11; footprint Switch_Keyboard_Kailh:SW_Kailh_Choc_V1V2_1.00u -> marbastlib-choc:SW_choc_v1_1u
- SW68: value COMMA -> EQUAL; footprint Switch_Keyboard_Kailh:SW_Kailh_Choc_V1V2_1.00u -> marbastlib-choc:SW_choc_v1_1u
- SW69: value DOT -> RBKT; footprint Switch_Keyboard_Kailh:SW_Kailh_Choc_V1V2_1.00u -> marbastlib-choc:SW_choc_v1_1u
- SW7: value F6 -> F1; footprint Switch_Keyboard_Kailh:SW_Kailh_Choc_V1V2_1.00u -> marbastlib-choc:SW_choc_v1_1u
- SW70: value MINUS -> NUHS; footprint Switch_Keyboard_Kailh:SW_Kailh_Choc_V1V2_1.00u -> marbastlib-choc:SW_choc_v1_1u
- SW71: value RSHIFT -> RSHFT; footprint Switch_Keyboard_Kailh:SW_Kailh_Choc_V1V2_1.75u -> marbastlib-choc:SW_choc_v1_1.75u
- SW72: value UP -> LEFT; footprint Switch_Keyboard_Kailh:SW_Kailh_Choc_V1V2_1.00u -> marbastlib-choc:SW_choc_v1_1u
- SW73: value END -> F12; footprint Switch_Keyboard_Kailh:SW_Kailh_Choc_V1V2_1.00u -> marbastlib-choc:SW_choc_v1_1u
- SW74: value LCTRL -> BSPC; footprint Switch_Keyboard_Kailh:SW_Kailh_Choc_V1V2_1.25u -> marbastlib-choc:SW_choc_v1_1u
- SW75: value LCMD -> ENTER; footprint Switch_Keyboard_Kailh:SW_Kailh_Choc_V1V2_1.25u -> Switch_Keyboard_Kailh:SW_Kailh_Choc_V1_ISOEnter
- SW76: value LALT -> UP; footprint Switch_Keyboard_Kailh:SW_Kailh_Choc_V1V2_1.25u -> marbastlib-choc:SW_choc_v1_1u
- SW77: value SPACE -> DOWN; footprint Switch_Keyboard_Kailh:SW_Kailh_Choc_V1V2_5.50u -> marbastlib-choc:SW_choc_v1_1u
- SW78: value RALT -> DEL; footprint Switch_Keyboard_Kailh:SW_Kailh_Choc_V1V2_1.25u -> marbastlib-choc:SW_choc_v1_1u
- SW79: value FN -> HOME; footprint Switch_Keyboard_Kailh:SW_Kailh_Choc_V1V2_1.25u -> marbastlib-choc:SW_choc_v1_1u
- SW8: value F7 -> 1; footprint Switch_Keyboard_Kailh:SW_Kailh_Choc_V1V2_1.00u -> marbastlib-choc:SW_choc_v1_1u
- SW80: value RCTRL -> PG_UP; footprint Switch_Keyboard_Kailh:SW_Kailh_Choc_V1V2_1.25u -> marbastlib-choc:SW_choc_v1_1u
- SW81: value LEFT -> PG_DN; footprint Switch_Keyboard_Kailh:SW_Kailh_Choc_V1V2_1.00u -> marbastlib-choc:SW_choc_v1_1u
- SW82: value DOWN -> END; footprint Switch_Keyboard_Kailh:SW_Kailh_Choc_V1V2_1.00u -> marbastlib-choc:SW_choc_v1_1u
- SW84: value Reset -> SW_SPST; footprint Button_Switch_THT:SW_PUSH_1P1T_6x3.5mm_H4.3_APEM_MJTP1243 -> Button_Switch_THT:SW_Slide_SPDT_Angled_CK_OS102011MA1Q
- SW9: value F8 -> Q; footprint Switch_Keyboard_Kailh:SW_Kailh_Choc_V1V2_1.00u -> marbastlib-choc:SW_choc_v1_1u
- moved SW29 293.1 mm to (51.3, 73.5)
- moved SW13 287.0 mm to (21.2, 103.6)
- moved SW27 284.5 mm to (36.2, 178.9)
- moved SW44 280.8 mm to (66.3, 148.8)
- moved SW28 275.4 mm to (51.3, 58.5)
- moved SW12 266.6 mm to (21.2, 88.6)
- moved SW26 261.8 mm to (36.2, 163.8)
- moved SW43 256.6 mm to (66.3, 133.7)
- moved SW58 250.2 mm to (96.4, 88.6)
- moved SW11 246.9 mm to (21.2, 73.5)
- moved SW9 245.8 mm to (6.13, 178.9)
- moved SW25 239.5 mm to (36.2, 148.8)
- moved J1 233.2 mm to (137.0, 176.4), turned to 0 degrees
- moved SW42 230.0 mm to (66.3, 118.7)
- moved SW10 228.0 mm to (21.2, 58.5)
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Connections:
- D1 pad 1: Net-(D1-K) -> P1.11
- D10 pad 1: Net-(D1-K) -> P0.02
- D11 pad 1: Net-(D1-K) -> P0.29
- D12 pad 1: Net-(D1-K) -> P0.31
- D13 pad 1: Net-(D1-K) -> P1.11
- D14 pad 1: Net-(D1-K) -> P1.13
- D15 pad 1: Net-(D15-K) -> P1.15
- D16 pad 1: Net-(D15-K) -> P0.02
- D17 pad 1: Net-(D15-K) -> P0.29
- D18 pad 1: Net-(D15-K) -> P0.31
- D19 pad 1: Net-(D15-K) -> P1.11
- D2 pad 1: Net-(D1-K) -> P1.13
- D20 pad 1: Net-(D15-K) -> P1.13
- D21 pad 1: Net-(D15-K) -> P1.15
- D22 pad 1: Net-(D15-K) -> P0.02
- D23 pad 1: Net-(D15-K) -> P0.29
- D24 pad 1: Net-(D15-K) -> P1.11
- D25 pad 1: Net-(D15-K) -> P1.13
- D26 pad 1: Net-(D15-K) -> P1.15
- D27 pad 1: Net-(D15-K) -> P0.02
- D28 pad 1: Net-(D15-K) -> P0.29
- D29 pad 1: Net-(D15-K) -> P1.13
- D3 pad 1: Net-(D1-K) -> P1.15
- D30 pad 1: Net-(D30-K) -> P1.15
- D31 pad 1: Net-(D30-K) -> P0.02
- D32 pad 1: Net-(D30-K) -> P0.29
- D33 pad 1: Net-(D30-K) -> P1.11
- D34 pad 1: Net-(D30-K) -> P1.13
- D35 pad 1: Net-(D30-K) -> P1.15
- D36 pad 1: Net-(D30-K) -> P0.02
- D37 pad 1: Net-(D30-K) -> P0.29
- D38 pad 1: Net-(D30-K) -> P0.31
- D39 pad 1: Net-(D30-K) -> P1.11
- D4 pad 1: Net-(D1-K) -> P0.02
- D40 pad 1: Net-(D30-K) -> P1.13
- D41 pad 1: Net-(D30-K) -> P1.15
- D42 pad 1: Net-(D30-K) -> P0.02
- D43 pad 1: Net-(D30-K) -> P0.29
- D44 pad 1: Net-(D44-K) -> P1.11
- D45 pad 1: Net-(D44-K) -> P1.13
- D46 pad 1: Net-(D44-K) -> P1.15
- D47 pad 1: Net-(D44-K) -> P0.02
- D48 pad 1: Net-(D44-K) -> P0.29
- D49 pad 1: Net-(D44-K) -> P1.11
- D5 pad 1: Net-(D1-K) -> P0.29
- D50 pad 1: Net-(D44-K) -> P1.13
- D51 pad 1: Net-(D44-K) -> P1.15
- D52 pad 1: Net-(D44-K) -> P0.02
- D53 pad 1: Net-(D44-K) -> P0.29
- D54 pad 1: Net-(D44-K) -> P0.31
- D55 pad 1: Net-(D44-K) -> P1.11
- D56 pad 1: Net-(D44-K) -> P1.13
- D57 pad 1: Net-(D44-K) -> P1.15
- D58 pad 1: Net-(D44-K) -> P0.02
- D59 pad 1: Net-(D59-K) -> P0.29
- D6 pad 1: Net-(D1-K) -> P0.31
- D60 pad 1: Net-(D59-K) -> P0.31
- D61 pad 1: Net-(D59-K) -> P1.11
- D62 pad 1: Net-(D59-K) -> P1.13
- D63 pad 1: Net-(D59-K) -> P1.15
- D64 pad 1: Net-(D59-K) -> P0.02
- D65 pad 1: Net-(D59-K) -> P0.29
- D66 pad 1: Net-(D59-K) -> P0.31
- D67 pad 1: Net-(D59-K) -> P1.11
- D68 pad 1: Net-(D59-K) -> P1.13
- D69 pad 1: Net-(D59-K) -> P1.15
- D7 pad 1: Net-(D1-K) -> P1.11
- D70 pad 1: Net-(D59-K) -> P0.02
- D71 pad 1: Net-(D59-K) -> P0.29
- D72 pad 1: Net-(D59-K) -> P0.31
- D73 pad 1: Net-(D59-K) -> P1.11
- D74 pad 1: Net-(D74-K) -> P1.13
- D75 pad 1: Net-(D74-K) -> P1.15
- D76 pad 1: Net-(D74-K) -> P0.29
- D77 pad 1: Net-(D74-K) -> P0.31
- D78 pad 1: Net-(D74-K) -> P1.11
- D79 pad 1: Net-(D74-K) -> P1.13
- D8 pad 1: Net-(D1-K) -> P1.13
- D80 pad 1: Net-(D74-K) -> P1.15
- D81 pad 1: Net-(D74-K) -> P0.02
- D82 pad 1: Net-(D74-K) -> P0.29
- D83 pad 1: Net-(D74-K) -> P0.31
- D9 pad 1: Net-(D1-K) -> P1.15
- J1 pad 1: Net-(U1-BATIN/P0.04) -> Net-(SW84-A)
- J1 pad 2: Net-(SW84-B) -> GND
- SW1 pad 1: Net-(SW1-A) -> P0.06
- SW10 pad 1: Net-(SW10-A) -> P0.08
- SW11 pad 1: Net-(SW11-A) -> P0.08
- SW12 pad 1: Net-(SW12-A) -> P0.08
- SW13 pad 1: Net-(SW13-A) -> P0.17
- SW14 pad 1: Net-(SW1-A) -> P0.17
- SW14 pad 2: Net-(D15-A) -> Net-(D14-A)
- SW15 pad 1: Net-(SW15-A) -> P0.17
- SW15 pad 2: Net-(D16-A) -> Net-(D15-A)
- SW16 pad 1: Net-(SW16-A) -> P0.17
- SW16 pad 2: Net-(D17-A) -> Net-(D16-A)
- SW17 pad 1: Net-(SW17-A) -> P0.17
- SW17 pad 2: Net-(D18-A) -> Net-(D17-A)
- SW18 pad 1: Net-(SW18-A) -> P0.17
- SW18 pad 2: Net-(D19-A) -> Net-(D18-A)
- SW19 pad 1: Net-(SW19-A) -> P0.20
- SW19 pad 2: Net-(D20-A) -> Net-(D19-A)
- SW2 pad 1: Net-(SW15-A) -> P0.06
- SW20 pad 1: Net-(SW20-A) -> P0.20
- SW20 pad 2: Net-(D21-A) -> Net-(D20-A)
- SW21 pad 1: Net-(SW21-A) -> P0.20
- SW21 pad 2: Net-(D22-A) -> Net-(D21-A)
- SW22 pad 1: Net-(SW22-A) -> P0.20
- SW22 pad 2: Net-(D23-A) -> Net-(D22-A)
- SW23 pad 1: Net-(SW23-A) -> P0.20
- SW23 pad 2: Net-(D24-A) -> Net-(D23-A)
- SW24 pad 1: Net-(SW10-A) -> P0.22
- SW24 pad 2: Net-(D25-A) -> Net-(D24-A)
- SW25 pad 1: Net-(SW11-A) -> P0.22
- SW25 pad 2: Net-(D26-A) -> Net-(D25-A)
- SW26 pad 1: Net-(SW12-A) -> P0.22
- SW26 pad 2: Net-(D27-A) -> Net-(D26-A)
- SW27 pad 1: Net-(SW13-A) -> P0.22
- SW27 pad 2: Net-(D28-A) -> Net-(D27-A)
- SW28 pad 1: Net-(SW28-A) -> P0.22
- SW28 pad 2: Net-(D29-A) -> Net-(D28-A)
- SW29 pad 1: Net-(D14-A) -> P0.24
- SW29 pad 2: Net-(SW28-A) -> Net-(D29-A)
- SW3 pad 1: Net-(SW16-A) -> P0.06
- SW30 pad 1: Net-(SW1-A) -> P0.24
- SW31 pad 1: Net-(SW15-A) -> P0.24
- SW32 pad 1: Net-(SW16-A) -> P0.24
- SW33 pad 1: Net-(SW17-A) -> P1.00
- SW34 pad 1: Net-(SW18-A) -> P1.00
- SW35 pad 1: Net-(SW19-A) -> P1.00
- SW36 pad 1: Net-(SW20-A) -> P1.00
- SW37 pad 1: Net-(SW21-A) -> P1.00
- SW38 pad 1: Net-(SW22-A) -> P1.00
- SW39 pad 1: Net-(SW23-A) -> P0.11
- SW4 pad 1: Net-(SW17-A) -> P0.06
- SW40 pad 1: Net-(SW10-A) -> P0.11
- SW41 pad 1: Net-(SW11-A) -> P0.11
- SW42 pad 1: Net-(SW12-A) -> P0.11
- SW43 pad 1: Net-(SW13-A) -> P0.11
- SW43 pad 2: Net-(D58-A) -> Net-(D43-A)
- SW44 pad 1: Net-(SW28-A) -> P1.04
- SW44 pad 2: Net-(D43-A) -> Net-(D44-A)
- SW45 pad 1: Net-(SW1-A) -> P1.04
- SW45 pad 2: Net-(D44-A) -> Net-(D45-A)
- SW46 pad 1: Net-(SW15-A) -> P1.04
- SW46 pad 2: Net-(D45-A) -> Net-(D46-A)
- SW47 pad 1: Net-(SW16-A) -> P1.04
- SW47 pad 2: Net-(D46-A) -> Net-(D47-A)
- SW48 pad 1: Net-(SW17-A) -> P1.04
- SW48 pad 2: Net-(D47-A) -> Net-(D48-A)
- SW49 pad 1: Net-(SW18-A) -> P1.06
- SW49 pad 2: Net-(D48-A) -> Net-(D49-A)
- SW5 pad 1: Net-(SW18-A) -> P0.06
- SW50 pad 1: Net-(SW19-A) -> P1.06
- SW50 pad 2: Net-(D49-A) -> Net-(D50-A)
- SW51 pad 1: Net-(SW20-A) -> P1.06
- SW51 pad 2: Net-(D50-A) -> Net-(D51-A)
- SW52 pad 1: Net-(SW21-A) -> P1.06
- SW52 pad 2: Net-(D51-A) -> Net-(D52-A)
- SW53 pad 1: Net-(SW22-A) -> P1.06
- SW53 pad 2: Net-(D52-A) -> Net-(D53-A)
- SW54 pad 1: Net-(SW23-A) -> P1.06
- SW54 pad 2: Net-(D53-A) -> Net-(D54-A)
- SW55 pad 1: Net-(SW10-A) -> P1.01
- SW55 pad 2: Net-(D54-A) -> Net-(D55-A)
- SW56 pad 1: Net-(SW11-A) -> P1.01
- SW56 pad 2: Net-(D55-A) -> Net-(D56-A)
- SW57 pad 1: Net-(SW12-A) -> P1.01
- SW57 pad 2: Net-(D56-A) -> Net-(D57-A)
- SW58 pad 1: Net-(SW28-A) -> P1.01
- SW58 pad 2: Net-(D57-A) -> Net-(D58-A)
- SW59 pad 1: Net-(SW1-A) -> P1.01
- SW6 pad 1: Net-(SW20-A) -> P0.06
- SW60 pad 1: Net-(SW15-A) -> P1.01
- SW61 pad 1: Net-(SW16-A) -> P1.02
- SW62 pad 1: Net-(SW17-A) -> P1.02
- SW63 pad 1: Net-(SW18-A) -> P1.02
- SW64 pad 1: Net-(SW19-A) -> P1.02
- SW65 pad 1: Net-(SW20-A) -> P1.02
- SW66 pad 1: Net-(SW21-A) -> P1.02
- SW67 pad 1: Net-(SW22-A) -> P1.07
- SW68 pad 1: Net-(SW23-A) -> P1.07
- SW69 pad 1: Net-(SW10-A) -> P1.07
- SW7 pad 1: Net-(SW21-A) -> P0.08
- SW70 pad 1: Net-(SW11-A) -> P1.07
- SW71 pad 1: Net-(SW12-A) -> P1.07
- SW72 pad 1: Net-(SW13-A) -> P1.07
- SW73 pad 1: Net-(SW28-A) -> P0.09
- SW74 pad 1: Net-(SW1-A) -> P0.09
- SW75 pad 1: Net-(SW15-A) -> P0.09
- SW76 pad 1: Net-(SW16-A) -> P0.09
- SW77 pad 1: Net-(SW20-A) -> P0.09
- SW78 pad 1: Net-(SW23-A) -> P0.10
- SW79 pad 1: Net-(SW10-A) -> P0.10
- SW8 pad 1: Net-(SW22-A) -> P0.08
- SW80 pad 1: Net-(SW11-A) -> P0.10
- SW81 pad 1: Net-(SW12-A) -> P0.10
- SW82 pad 1: Net-(SW13-A) -> P0.10
- SW83 pad 1: Net-(SW28-A) -> P0.10
- SW84 pad 2: Net-(SW84-B) -> BATIN
- SW9 pad 1: Net-(SW23-A) -> P0.08
- U1 pad 1: Net-(SW1-A) -> P0.06
- U1 pad 10: Net-(SW21-A) -> P0.11
- U1 pad 11: Net-(SW22-A) -> P1.04
- U1 pad 12: Net-(SW23-A) -> P1.06
- U1 pad 13: Net-(SW13-A) -> P0.09
- U1 pad 14: Net-(SW28-A) -> P0.10
- U1 pad 15: Net-(D1-K) -> P1.11
- U1 pad 16: Net-(D15-K) -> P1.13
- U1 pad 17: Net-(D30-K) -> P1.15
- U1 pad 18: Net-(D44-K) -> P0.02
- U1 pad 19: Net-(D59-K) -> P0.29
- U1 pad 2: Net-(SW15-A) -> P0.08
- U1 pad 20: Net-(D74-K) -> P0.31
- U1 pad 22: Net-(SW84-A) -> unconnected-(U1-RST-Pad22)
- U1 pad 23: Net-(SW84-B) -> GND
- U1 pad 24: Net-(U1-BATIN/P0.04) -> BATIN
- U1 pad 3: Net-(SW84-B) -> GND
- U1 pad 31: Net-(SW10-A) -> P1.01
- U1 pad 32: Net-(SW11-A) -> P1.02
- U1 pad 33: Net-(SW12-A) -> P1.07
- U1 pad 4: Net-(SW84-B) -> GND
- U1 pad 5: Net-(SW16-A) -> P0.17
- U1 pad 6: Net-(SW17-A) -> P0.20
- U1 pad 7: Net-(SW18-A) -> P0.22
- U1 pad 8: Net-(SW19-A) -> P0.24
- U1 pad 9: Net-(SW20-A) -> P1.00
Routing:
- net Net-(SW1-A): track 400.9 -> 0.00 mm
- net Net-(D74-K): track 386.0 -> 0.00 mm
- net Net-(SW15-A): track 373.1 -> 0.00 mm
- net Net-(D59-K): track 368.1 -> 0.00 mm
- net Net-(D44-K): track 350.4 -> 0.00 mm
- net Net-(SW16-A): track 347.1 -> 0.00 mm
- net Net-(D30-K): track 335.3 -> 0.00 mm
- net Net-(SW17-A): track 303.9 -> 0.00 mm
- net Net-(D15-K): track 291.5 -> 0.00 mm
- net Net-(SW18-A): track 284.5 -> 0.00 mm
- net Net-(D1-K): track 274.7 -> 0.00 mm
- net Net-(SW20-A): track 271.1 -> 0.00 mm
- net Net-(SW19-A): track 258.7 -> 0.00 mm
- net Net-(SW21-A): track 228.7 -> 0.00 mm
- net Net-(SW22-A): track 206.8 -> 0.00 mm
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Other:
- board outline removed
- board text removed: "${REFERENCE}"
- board text removed: "002"
- board text removed: "006"
- board text removed: "008"
- board text removed: "010"
- board text removed: "017"
- board text removed: "020"
- board text removed: "022"
- board text removed: "024"
- board text removed: "029"
- board text removed: "031"
- board text removed: "100"
- board text removed: "104"
- board text removed: "111"
- board text removed: "113"
- board text removed: "115"
- board text removed: "GND"
- board text removed: "RAW"
- board text removed: "RST"
- board text removed: "VCC"
- board text removed: "nice!nano"

Commit message: Added spacings to keycaps for easier alignment
Parts:
- added SW85: RESET, Button_Switch_THT:SW_PUSH_1P1T_6x3.5mm_H4.3_APEM_MJTP1243, F.Cu at (64.4, 199.8)
- J1: value S2B-PH-K-SLFSN -> BATTERY
- SW1, SW10, SW11, SW13, SW14, SW15, SW16, SW17, SW19, SW2, SW20, SW21, SW22, SW23, SW24, SW25, SW26, SW27, SW28, SW29, SW30, SW31, SW32, SW33, SW34, SW35, SW36, SW37, SW39, SW40, SW41, SW42, SW43, SW44, SW45, SW46, SW47, SW48, SW49, SW50, SW51, SW52, SW53, SW55, SW56, SW57, SW58, SW59, SW61, SW62, SW63, SW64, SW65, SW67, SW68, SW69, SW7, SW70, SW72, SW73, SW74, SW76, SW77, SW78, SW79, SW8, SW80, SW81, SW82, SW83, SW9: footprint marbastlib-choc:SW_choc_v1_1u -> Switch_Keyboard_Kailh:SW_Kailh_Choc_V1_1.00u_Spacing
- SW12, SW18, SW54, SW60, SW66: footprint marbastlib-choc:SW_choc_v1_1.25u -> Switch_Keyboard_Kailh:SW_Kailh_Choc_V1_1.25u_Spacing
- SW3: footprint marbastlib-choc:SW_choc_v1_1.5u -> Switch_Keyboard_Kailh:SW_Kailh_Choc_V1_1.50u_Spacing
- SW38: footprint Switch_Keyboard_Kailh:SW_Kailh_Choc_V1_6.00u -> Switch_Keyboard_Kailh:SW_Kailh_Choc_V1_6.00u_Spacing
- SW4: footprint marbastlib-choc:SW_choc_v1_1.75u -> Switch_Keyboard_Kailh:SW_Kailh_Choc_V1_1.75u_Spacing
- SW5, SW6: footprint marbastlib-choc:SW_choc_v1_1.25u -> Switch_Keyboard_Kailh:SW_Kailh_Choc_V1_1.50u_Spacing
- SW71: footprint marbastlib-choc:SW_choc_v1_1.75u -> Switch_Keyboard_Kailh:SW_Kailh_Choc_V1_1.00u_Spacing
- SW75: footprint Switch_Keyboard_Kailh:SW_Kailh_Choc_V1_ISOEnter -> Switch_Keyboard_Kailh:SW_Kailh_Choc_V1_ISOEnter_Spacing
- SW84: value SW_SPST -> POWER
- moved SW18 222.5 mm to (191.9, 36.1)
- moved SW3 192.3 mm to (176.9, 176.8)
- moved SW6 190.0 mm to (176.9, 217.0)
- moved SW5 187.9 mm to (176.9, 196.9)
- moved SW12 185.5 mm to (191.9, 16.0)
- moved SW75 176.5 mm to (-34.0, 160.2)
- moved SW54 154.3 mm to (191.9, 56.2)
- moved U1 130.2 mm to (46.5, 196.4)
- moved SW4 119.0 mm to (45.1, 216.1)
- moved D14 118.6 mm to (110.1, 214.7)
- moved D21 118.6 mm to (120.9, 179.2)
- moved D26 118.6 mm to (120.9, 196.9)
- moved D31 118.6 mm to (120.9, 214.7)
- moved D38 118.6 mm to (131.7, 179.2)
- moved D4 118.6 mm to (110.1, 179.2)
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Connections:
- U1 pad 21: unconnected-(U1-VCC-Pad21) -> RESET
- U1 pad 22: unconnected-(U1-RST-Pad22) -> GND

Commit message: Started positioning switches
Parts:
- moved SW3 293.7 mm to (-12.0, -48.0)
- moved SW7 145.2 mm to (11.5, -89.0)
- moved SW9 144.4 mm to (11.5, -48.0)
- moved SW8 143.4 mm to (2.50, -67.0)
- moved SW1 107.9 mm to (-16.5, -89.0)
- moved SW2 106.1 mm to (-16.5, -67.0)
- moved SW38 25.1 mm to (28.5, 174.0)

Commit message: Finished positioning switches
Parts:
- SW37: footprint Switch_Keyboard_Kailh:SW_Kailh_Choc_V1_1.00u_Spacing -> Switch_Keyboard_Kailh:SW_Kailh_Choc_V1_5.50u_Spacing
- SW38: footprint Switch_Keyboard_Kailh:SW_Kailh_Choc_V1_6.00u_Spacing -> Switch_Keyboard_Kailh:SW_Kailh_Choc_V1_5.50u_Spacing
- SW71: footprint Switch_Keyboard_Kailh:SW_Kailh_Choc_V1_1.00u_Spacing -> Switch_Keyboard_Kailh:SW_Kailh_Choc_V1_1.50u_Spacing
- moved U1 356.6 mm to (260.2, -89.0), turned to 180 degrees
- moved SW75 344.0 mm to (246.0, -39.5)
- moved SW85 335.2 mm to (243.0, -83.8), turned to 90 degrees
- moved SW6 281.0 mm to (-12.0, 9.00)
- moved SW5 280.2 mm to (-12.0, -10.0)
- moved SW13 258.1 mm to (30.5, -90.0)
- moved SW4 251.1 mm to (-9.75, -29.0)
- moved SW39 250.4 mm to (111.5, -90.0)
- moved SW73 240.7 mm to (230.5, -90.0)
- moved SW74 238.0 mm to (230.5, -67.0)
- moved SW55 235.6 mm to (173.5, -90.0)
- moved SW56 232.8 mm to (173.5, -67.0)
- moved SW22 227.8 mm to (54.0, -29.0)
- moved SW30 208.3 mm to (87.5, -48.0)
- moved SW29 205.8 mm to (78.5, -67.0)
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
Commit message: Started pulling lanes
Parts:
- D1, D10, D11, D12, D13, D14, D15, D16, D17, D18, D19, D2, D20, D21, D22, D23, D24, D25, D26, D27, D28, D29, D3, D30, D31, D32, D33, D34, D35, D36, D37, D38, D39, D4, D40, D41, D42, D43, D44, D45, D46, D47, D48, D49, D5, D50, D51, D52, D53, D54, D55, D56, D57, D58, D59, D6, D60, D61, D62, D63, D64, D65, D66, D67, D68, D69, D7, D70, D71, D72, D73, D74, D75, D76, D77, D78, D79, D8, D80, D81, D82, D83, D9, J1, SW84: moved to B.Cu
- SW37: footprint Switch_Keyboard_Kailh:SW_Kailh_Choc_V1_5.50u_Spacing -> Switch_Keyboard_Kailh:SW_Kailh_Choc_V1_1.00u_Spacing
- moved J1 427.7 mm to (269.6, -92.0), turned to -90 degrees
- moved SW84 409.8 mm to (276.0, -83.0), turned to -90 degrees
- moved D67 394.7 mm to (221.0, -86.2), turned to 90 degrees
- moved D33 387.0 mm to (102.0, -86.2), turned to 90 degrees
- moved D49 384.1 mm to (159.0, -86.2), turned to 90 degrees
- moved D13 382.2 mm to (40.0, -86.2), turned to 90 degrees
- moved D79 376.2 mm to (264.2, -76.5)
- moved D68 375.6 mm to (221.0, -63.2), turned to 90 degrees
- moved D61 370.3 mm to (202.0, -86.2), turned to 90 degrees
- moved D34 367.3 mm to (107.0, -63.2), turned to 90 degrees
- moved D7 365.4 mm to (21.0, -86.2), turned to 90 degrees
- moved D44 365.4 mm to (140.0, -86.2), turned to 90 degrees
- moved D50 365.1 mm to (164.0, -63.2), turned to 90 degrees
- moved D14 364.9 mm to (31.0, -63.2), turned to 90 degrees
- moved D80 361.1 mm to (263.0, -57.5)
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Routing:
- net P0.06: track 0.00 -> 292.2 mm
- net P0.08: track 0.00 -> 261.3 mm
- net P0.17: track 0.00 -> 234.4 mm
- net P0.20: track 0.00 -> 212.5 mm
- net P0.24: track 0.00 -> 195.7 mm
- net P0.22: track 0.00 -> 192.5 mm
- net P1.00: track 0.00 -> 162.8 mm
- net P0.11: track 0.00 -> 140.9 mm
- net P1.04: track 0.00 -> 119.0 mm
- net P1.06: track 0.00 -> 97.2 mm
- net P1.01: track 0.00 -> 85.8 mm
- net P1.02: track 0.00 -> 65.8 mm
- net GND: track 0.00 -> 49.6 mm
- net P1.07: track 0.00 -> 45.7 mm
- net P0.10: track 0.00 -> 27.6 mm
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Other:
- board outline added: 304.5 x 119 mm

Commit message: Made Column traces
Parts:
- moved J1 205.3 mm to (367.8, 88.2), turned to 90 degrees
- moved D1 200.8 mm to (85.5, 92.3)
- moved D10 200.8 mm to (117.5, 153.3)
- moved D11 200.8 mm to (113.0, 172.3)
- moved D12 200.8 mm to (117.5, 191.3)
- moved D13 200.8 mm to (132.0, 92.3)
- moved D14 200.8 mm to (123.0, 115.3)
- moved D15 200.8 mm to (132.0, 134.3)
- moved D16 200.8 mm to (136.5, 153.3)
- moved D17 200.8 mm to (132.0, 172.3)
- moved D18 200.8 mm to (141.0, 191.3)
- moved D19 200.8 mm to (151.0, 92.3)
- moved D2 200.8 mm to (85.0, 115.3)
- moved D20 200.8 mm to (142.0, 115.3)
- moved D21 200.8 mm to (151.0, 134.3)
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Connections:
- J1 pad 1: Net-(SW84-A) -> Net-(SW84-B)
- SW84 pad 1: Net-(SW84-A) -> unconnected-(SW84-A-Pad1)
- SW84 pad 2: BATIN -> Net-(SW84-B)
- SW84 pad 3: (no net) -> BATIN
- U1 pad 21: RESET -> unconnected-(U1-VCC-Pad21)
- U1 pad 22: GND -> RESET
Routing:
- net P0.17: track 234.4 -> 348.0 mm
- net P1.00: track 162.8 -> 275.1 mm
- net P0.09: track 20.5 -> 132.5 mm
- net P0.08: track 261.3 -> 373.1 mm
- net P1.06: track 97.2 -> 207.5 mm
- net P0.06: track 292.2 -> 399.0 mm
- net P1.07: track 45.7 -> 152.3 mm
- net P1.02: track 65.8 -> 172.1 mm
- net P1.01: track 85.8 -> 190.2 mm
- net P0.20: track 212.5 -> 304.3 mm
- net P0.11: track 140.9 -> 231.1 mm
- net P1.04: track 119.0 -> 209.2 mm
- net P0.22: track 192.5 -> 282.5 mm
- net P0.10: track 27.6 -> 110.3 mm
- net P0.24: track 195.7 -> 256.0 mm
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
Commit message: Thinking about moving battery and connector below spacebar
Parts:
- added REF**: 401030 Lipo Battery Size, Library:401030 Lipo Battery Size, B.Cu at (165.0, 190.0)
- moved SW85 0.40 mm to (334.1, 101.2)
Routing:
- net P0.31: track 0.00 -> 354.2 mm
- net P0.29: track 0.00 -> 336.5 mm
- net P1.15: track 0.00 -> 310.2 mm
- net P0.02: track 0.00 -> 308.1 mm
- net P1.13: track 0.00 -> 284.7 mm
- net P1.11: track 0.00 -> 284.0 mm
- net Net-(D38-A): track 45.0 -> 0.01 mm
- net Net-(D18-A): track 6.75 -> 51.7 mm
- net P0.24: track 256.0 -> 263.9 mm, vias 0 -> 1

Commit message: Finished most work, now screwsholes are missing
Parts:
- moved J1 176.5 mm to (222.4, 188.5)
- moved REF** 11.4 mm to (176.4, 190.2)
Routing:
- net Net-(SW84-B): track 10.4 -> 233.9 mm, vias 0 -> 1
- net GND: track 56.8 -> 184.6 mm, vias 0 -> 1
- net Net-(D38-A): track 0.01 -> 45.7 mm
- net Net-(D18-A): track 51.7 -> 6.75 mm
- net P0.09: track 132.5 -> 138.0 mm
- net P0.02: track 308.1 -> 308.8 mm
- added copper zone on B.Cu, net GND
Other:
- board text added: "AC_K1_v1"
