File: AC-K1-v1.kicad_pcb (KiCad board)
At the start: 2 copper layers, 304.5 x 119 mm, 171 parts, among them J1 BATTERY, SW1 ESC, SW10 A, SW11 BSLH, SW12 LCMD, SW13 F2, SW14 2, SW15 W, SW16 S, SW17 Z, SW18 LALT, SW19 F3, SW2 GRAVE, SW20 3, SW21 E, SW22 D, SW23 X, SW24 F4, SW25 4, SW26 R, SW27 F, SW28 C, SW29 5, SW3 TAB, SW30 T, SW31 G, SW32 V, SW33 F5, SW34 6, SW35 Y, SW36 H, SW37 B, SW38 SPACE, SW39 F6, SW4 LCTRL, SW40 7, SW41 U, SW42 J, SW43 N, SW44 F7, SW45 8, SW46 I, SW47 K, SW48 M, SW49 F8, SW5 LSHIFT, SW50 9, SW51 O, SW52 L, SW53 COMMA, SW54 RALT, SW55 F9, SW56 0, SW57 P, SW58 SEMI, SW59 DOT, SW6 LCTRL, SW60 FN, SW61 F10, SW62 MINUS, SW63 LBKT, SW64 SQT, SW65 FSLH, SW66 RCTRL, SW67 F11, SW68 EQUAL, SW69 RBKT, SW7 F1, SW70 NUHS, SW71 RSHFT, SW72 LEFT, SW73 F12, SW74 BSPC, SW75 ENTER, SW76 UP, SW77 DOWN, SW78 DEL, SW79 HOME, SW8 1, SW80 PG_UP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

Commit message: Made small changes in routing.
Parts:
- moved J1 166.9 mm to (357.9, 91.0)
- moved REF** 154.6 mm to (304.4, 103.5)
- moved SW84 5.80 mm to (367.2, 89.0)
Routing:
- net Net-(SW84-B): track 233.9 -> 9.30 mm, vias 1 -> 0
- net GND: track 184.6 -> 0.02 mm, vias 1 -> 0
- net BATIN: track 2.94 -> 5.82 mm

Commit message: PCB Almost finished
Parts:
- added 1: MountingHole_2.7mm_M2.5_with_spacer, Library:MountingHole_2.7mm_M2.5_with_spacer, F.Cu at (90.5, 82.5)
- added 10: MountingHole_2.7mm_M2.5_with_spacer, Library:MountingHole_2.7mm_M2.5_with_spacer, F.Cu at (92.0, 122.5)
- added 11: MountingHole_2.7mm_M2.5_with_spacer, Library:MountingHole_2.7mm_M2.5_with_spacer, F.Cu at (346.5, 125.5)
- added 12: MountingHole_2.7mm_M2.5_with_spacer, Library:MountingHole_2.7mm_M2.5_with_spacer, F.Cu at (69.0, 130.5)
- added 13: MountingHole_2.7mm_M2.5_with_spacer, Library:MountingHole_2.7mm_M2.5_with_spacer, F.Cu at (327.0, 132.5)
- added 14: MountingHole_2.7mm_M2.5_with_spacer, Library:MountingHole_2.7mm_M2.5_with_spacer, F.Cu at (95.5, 142.0)
- added 15: MountingHole_2.7mm_M2.5_with_spacer, Library:MountingHole_2.7mm_M2.5_with_spacer, F.Cu at (346.0, 154.5)
- added 16: MountingHole_2.7mm_M2.5_with_spacer, Library:MountingHole_2.7mm_M2.5_with_spacer, F.Cu at (306.0, 160.5)
- added 17: MountingHole_2.7mm_M2.5_with_spacer, Library:MountingHole_2.7mm_M2.5_with_spacer, F.Cu at (69.0, 163.5)
- added 18: MountingHole_2.7mm_M2.5_with_spacer, Library:MountingHole_2.7mm_M2.5_with_spacer, F.Cu at (328.0, 176.0)
- added 19: MountingHole_2.7mm_M2.5_with_spacer, Library:MountingHole_2.7mm_M2.5_with_spacer, F.Cu at (140.5, 179.5)
- added 2: MountingHole_2.7mm_M2.5_with_spacer, Library:MountingHole_2.7mm_M2.5_with_spacer, F.Cu at (361.6, 88.7)
- added 20: MountingHole_2.7mm_M2.5_with_spacer, Library:MountingHole_2.7mm_M2.5_with_spacer, F.Cu at (180.0, 179.5)
- added 21: MountingHole_2.7mm_M2.5_with_spacer, Library:MountingHole_2.7mm_M2.5_with_spacer, F.Cu at (212.5, 179.5)
- added 22: MountingHole_2.7mm_M2.5_with_spacer, Library:MountingHole_2.7mm_M2.5_with_spacer, F.Cu at (241.5, 179.5)
- added 23: MountingHole_2.7mm_M2.5_with_spacer, Library:MountingHole_2.7mm_M2.5_with_spacer, F.Cu at (288.0, 179.5)
- added 24: MountingHole_2.7mm_M2.5_with_spacer, Library:MountingHole_2.7mm_M2.5_with_spacer, F.Cu at (69.0, 194.0)
- added 25: MountingHole_2.7mm_M2.5_with_spacer, Library:MountingHole_2.7mm_M2.5_with_spacer, F.Cu at (169.5, 194.0)
- added 26: MountingHole_2.7mm_M2.5_with_spacer, Library:MountingHole_2.7mm_M2.5_with_spacer, F.Cu at (212.5, 193.5)
- added 27: MountingHole_2.7mm_M2.5_with_spacer, Library:MountingHole_2.7mm_M2.5_with_spacer, F.Cu at (328.0, 160.0)
- added 3: MountingHole_2.7mm_M2.5_with_spacer, Library:MountingHole_2.7mm_M2.5_with_spacer, F.Cu at (69.0, 100.0)
- added 4: MountingHole_2.7mm_M2.5_with_spacer, Library:MountingHole_2.7mm_M2.5_with_spacer, F.Cu at (107.0, 100.0)
- added 5: MountingHole_2.7mm_M2.5_with_spacer, Library:MountingHole_2.7mm_M2.5_with_spacer, F.Cu at (147.0, 100.0)
- added 6: MountingHole_2.7mm_M2.5_with_spacer, Library:MountingHole_2.7mm_M2.5_with_spacer, F.Cu at (195.0, 100.0)
- added 7: MountingHole_2.7mm_M2.5_with_spacer, Library:MountingHole_2.7mm_M2.5_with_spacer, F.Cu at (237.0, 100.0)
- added 8: MountingHole_2.7mm_M2.5_with_spacer, Library:MountingHole_2.7mm_M2.5_with_spacer, F.Cu at (275.0, 100.0)
- added 9: MountingHole_2.7mm_M2.5_with_spacer, Library:MountingHole_2.7mm_M2.5_with_spacer, F.Cu at (327.5, 100.0)
- added REF**: PCB-Support, Library:PCB-Support, B.Cu at (104.5, 178.0)
- added REF**: PCB-Support, Library:PCB-Support, B.Cu at (236.5, 159.0)
- added REF**: PCB-Support, Library:PCB-Support, B.Cu at (74.5, 140.0)
- added REF**: PCB-Support, Library:PCB-Support, B.Cu at (78.5, 121.0)
- added REF**: PCB-Support, Library:PCB-Support, B.Cu at (87.5, 99.5)
- added REF**: PCB-Support, Library:PCB-Support, B.Cu at (174.5, 89.5)
- added REF**: PCB-Support, Library:PCB-Support, B.Cu at (173.5, 100.0)
- added REF**: PCB-Support, Library:PCB-Support, B.Cu at (341.5, 178.0)
- added REF**: PCB-Support, Library:PCB-Support, B.Cu at (158.5, 121.0)
- added REF**: PCB-Support, Library:PCB-Support, B.Cu at (274.5, 159.0)
- added REF**: PCB-Support, Library:PCB-Support, B.Cu at (201.5, 140.0)
- added REF**: PCB-Support, Library:PCB-Support, B.Cu at (79.5, 178.0)
- added REF**: PCB-Support, Library:PCB-Support, B.Cu at (253.5, 100.0)
- added REF**: PCB-Support, Library:PCB-Support, B.Cu at (128.5, 99.5)
- added REF**: PCB-Support, Library:PCB-Support, B.Cu at (239.5, 140.0)
- added REF**: PCB-Support, Library:PCB-Support, B.Cu at (198.5, 159.0)
- added REF**: PCB-Support, Library:PCB-Support, B.Cu at (216.0, 99.5)
- added REF**: PCB-Support, Library:PCB-Support, B.Cu at (308.5, 178.0)
- added REF**: PCB-Support, Library:PCB-Support, B.Cu at (315.5, 140.0)
- added REF**: PCB-Support, Library:PCB-Support, B.Cu at (163.5, 140.0)
- added REF**: PCB-Support, Library:PCB-Support, B.Cu at (264.0, 178.0)
- added REF**: PCB-Support, Library:PCB-Support, B.Cu at (326.0, 121.0)
- added REF**: PCB-Support, Library:PCB-Support, B.Cu at (120.5, 121.0)
- added REF**: PCB-Support, Library:PCB-Support, B.Cu at (277.5, 140.0)
- added REF**: PCB-Support, Library:PCB-Support, B.Cu at (253.5, 121.0)
- added REF**: PCB-Support, Library:PCB-Support, B.Cu at (255.5, 89.5)
- added REF**: PCB-Support, Library:PCB-Support, B.Cu at (196.5, 121.0)
- added REF**: PCB-Support, Library:PCB-Support, B.Cu at (122.5, 159.0)
- added REF**: PCB-Support, Library:PCB-Support, B.Cu at (291.5, 121.0)
- added REF**: PCB-Support, Library:PCB-Support, B.Cu at (160.5, 159.0)
- added REF**: PCB-Support, Library:PCB-Support, B.Cu at (125.5, 140.0)
- moved J1 1.34 mm to (356.6, 91.0)
- renumbered REF** to Battery1
Routing:
- net Net-(SW84-B): track 9.30 -> 10.6 mm
- net P0.24: track 263.9 -> 265.1 mm
Other:
- board size 304.5 x 119 mm -> 304.5 x 119.5 mm

Commit message: Adjusted screws
Parts:
- added REF**: MountingHole_2.7mm_M2.5_with_spacer, Library:MountingHole_2.7mm_M2.5_with_spacer, F.Cu at (92.0, 178.5)
- moved 24 1.77 mm to (69.2, 192.2)
- moved 3 1.25 mm to (70.2, 100.0)
- moved 25 0.45 mm to (169.5, 193.6)
- moved 12 0.25 mm to (69.2, 130.5)
- moved 17 0.25 mm to (69.2, 163.5)
Changed lines of the file:
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@@
 	(footprint "Library:MountingHole_2.7mm_M2.5_with_spacer"
 		(layer "F.Cu")
-		(at 169.5 194)
+		(at 169.5 193.55)
 		(descr "Mounting Hole 2.7mm, no annular, M2.5")
 		(tags "mounting hole 2.7mm no annular m2.5")
@@
 		)
 		(fp_text user "${REFERENCE}"
-			(at 0 0 0)
+			(at -0.06 -0.03 0)
 			(layer "F.Fab")
 			(effects
@@
 	(footprint "Library:MountingHole_2.7mm_M2.5_with_spacer"
 		(layer "F.Cu")
-		(at 69 130.5)
+		(at 69.25 130.5)
 		(descr "Mounting Hole 2.7mm, no annular, M2.5")
 		(tags "mounting hole 2.7mm no annular m2.5")
@@
 		)
 	)
+	(footprint "Library:MountingHole_2.7mm_M2.5_with_spacer"
+		(layer "F.Cu")
+		(at 92 178.5)
+		(descr "Mounting Hole 2.7mm, no annular, M2.5")
+		(tags "mounting hole 2.7mm no annular m2.5")
+		(property "Reference" "REF**"
+			(at 0 -3.7 0)
+			(layer "F.SilkS")
+			(effects
+				(font
+					(size 1 1)
+					(thickness 0.15)
+				)
+			)
+		)
+		(property "Value" "MountingHole_2.7mm_M2.5_with_spacer"
+			(at 0 3.7 0)
+			(layer "F.Fab")
+			(hide yes)
+			(effects
+				(font
+					(size 1 1)
+					(thickness 0.15)
+				)
+			)
+		)
+		(property "Footprint" "Library:MountingHole_2.7mm_M2.5_with_spacer"
+			(at 0 0 0)
+			(unlocked yes)
+			(layer "F.Fab")
+			(hide yes)
+			(effects
+				(font
+					(size 1.27 1.27)
+					(thickness 0.15)
+				)
+			)
+		)
+		(property "Datasheet" ""
+			(at 0 0 0)
+			(unlocked yes)
+			(layer "F.Fab")
+			(hide yes)
+			(effects
+				(font
+					(size 1.27 1.27)
+					(thickness 0.15)
+				)
+			)
+		)
+		(property "Description" ""
+			(at 0 0 0)
+			(unlocked yes)
+			(layer "F.Fab")
+			(hide yes)
+			(effects
+				(font
+					(size 1.27 1.27)
+					(thickness 0.15)
+				)
+			)
+		)
+		(attr exclude_from_pos_files exclude_from_bom)
+		(fp_circle
+			(center 0 0)
+			(end 2.7 0)
+			(stroke
+				(width 0.15)
+				(type solid)
+			)
+			(fill none)
+			(layer "Cmts.User")
+		)
+		(fp_circle
+			(center 0 0)
+			(end 2.9 0)
+			(stroke
+				(width 0.05)
+				(type default)
+			)
+			(fill none)
+			(layer "B.CrtYd")
+		)
+		(fp_circle
+			(center 0 0)
+			(end 2.95 0)
+			(stroke
+				(width 0.05)
+				(type solid)
+			)
+			(fill none)
+			(layer "F.CrtYd")
+		)
+		(fp_text user "${REFERENCE}"
+			(at 0 0 0)
+			(layer "F.Fab")
+			(effects
+				(font
+					(size 1 1)
+					(thickness 0.15)
+				)
+			)
+		)
+		(pad "" np_thru_hole circle
+			(at 0 0)
+			(size 2.7 2.7)
+			(drill 2.7)
+			(layers "*.Cu" "*.Mask")
+		)
+		(model "${KIPRJMOD}/Library.pretty/3D-Models/PCB-Screw-Spacer.step"
+			(offset
+				(xyz 0 0 -4.5)
+			)
+			(scale
+				(xyz 1 1 1)
+			)
+			(rotate
+				(xyz 0 0 0)
+			)
+		)
+	)
 	(footprint "Switch_Keyboard_Kailh:SW_Kailh_Choc_V1_1.00u_Spacing"
 		(locked yes)
@@
 	(footprint "Library:MountingHole_2.7mm_M2.5_with_spacer"
 		(layer "F.Cu")
-		(at 69 100)
+		(at 70.25 100)
 		(descr "Mounting Hole 2.7mm, no annular, M2.5")
 		(tags "mounting hole 2.7mm no annular m2.5")
@@
 	(footprint "Library:MountingHole_2.7mm_M2.5_with_spacer"
 		(layer "F.Cu")
-		(at 69 163.5)
+		(at 69.25 163.5)
 		(descr "Mounting Hole 2.7mm, no annular, M2.5")
 		(tags "mounting hole 2.7mm no annular m2.5")
@@
 	(footprint "Library:MountingHole_2.7mm_M2.5_with_spacer"
 		(layer "F.Cu")
-		(at 69 194)
+		(at 69.25 192.25)
 		(descr "Mounting Hole 2.7mm, no annular, M2.5")
 		(tags "mounting hole 2.7mm no annular m2.5")

Commit message: Added top ground zone and changed screw positions
Parts:
- removed 12, 17, 24, 25, 26, 3: MountingHole_2.7mm_M2.5_with_spacer, Library:MountingHole_2.7mm_M2.5_with_spacer
- added REF**: PCB-Support, Library:PCB-Support, B.Cu at (213.0, 193.5)
- added REF**: PCB-Support, Library:PCB-Support, B.Cu at (169.5, 193.5)
- added REF**: PCB-Support, Library:PCB-Support, B.Cu at (69.0, 187.5)
- added REF**: PCB-Support, Library:PCB-Support, B.Cu at (69.0, 168.5)
- added REF**: PCB-Support, Library:PCB-Support, B.Cu at (69.0, 129.0)
- moved REF** 11.5 mm to (76.0, 100.0)
- moved 1 6.02 mm to (90.0, 88.5)
- moved REF** 1.50 mm to (80.0, 121.0)
- moved 50 1.00 mm to (92.0, 179.5)
- moved 15 0.50 mm to (346.5, 154.5)
- moved 27 0.50 mm to (328.0, 160.5)
- renumbered REF** to 50
Routing:
- added copper zone on F.Cu, net GND
